Commit message: feat(sim): articulated rocker-bogie suspension (passive rocker + bogie per side)
Replaces the rigid chassis with the real passive linkage: per side a rocker
(revolute, axis Y) on the body carrying the front wheel + a bogie carrying mid/
rear wheels. Pure passive damped joints; wheels still measured-accurate at zero
angle. Cross-body differential omitted (closed loop; noted).

Co-Authored-By: Claude Opus 4.8 <noreply@anthropic.com>

File: src/friday_description/urdf/mark1.urdf.xacro (robot description, xacro)
@@ -1,56 +1,57 @@
 <?xml version="1.0"?>
 <!--
-  Mark 1 — Stage 1 sim model (first-light).
-  Geometry is measured directly from the scaled-Perseverance model
-  (Mechanics/reference-models/perseverance/mark1_sim_spec.md), expressed in the
-  ROS REP-103 frame: +X forward, +Y left, +Z up. Wheels spin about Y.
-  First-light scope: a RIGID six-wheel chassis (wheels mounted straight to the
-  body) so the sim pipeline is proven to spawn / stand / drive. The articulated
-  rocker-bogie pivots (passive revolute rocker + bogie per side) are the next
-  refinement — see the TODO at the bottom. Drive is skid/differential via
-  gz_ros2_control + diff_drive_controller (left 3 wheels / right 3 wheels).
+  Mark 1 — Stage 1 sim model: articulated six-wheel ROCKER-BOGIE.
+  Frame: ROS REP-103 (+X forward, +Y left, +Z up). Wheels spin about Y.
+  Geometry measured from the scaled-Perseverance model
+  (Mechanics/reference-models/perseverance/mark1_sim_spec.md). At zero suspension
+  angle every wheel sits exactly at its measured (x, y) on the axle plane (z 0).
+  Per side: a PASSIVE rocker (revolute, axis Y) pivots on the body and carries the
+  front wheel + a PASSIVE bogie (revolute, axis Y); the bogie carries the mid and
+  rear wheels. Pure passive damped joints (no springs) — the rocker-bogie levels by
+  geometry + gravity, like the real rover. The 6 wheels are velocity-driven via
+  gz_ros2_control + diff_drive_controller (skid steer, left 3 / right 3).
+  Simplification (noted): the cross-body differential bar (a closed kinematic loop)
+  is omitted — URDF is a tree. On flat/symmetric ground the body settles level; on
+  rough ground it rolls slightly more than the real differential-coupled rover.
 -->
 <robot name="mark1" xmlns:xacro="http://www.ros.org/wiki/xacro">
   <xacro:arg name="controllers_yaml" default=""/>
-  <!-- ===== measured parameters (metres / kg) ===== -->
+  <!-- ===== measured parameters (m / kg) ===== -->
   <xacro:property name="wheel_radius" value="0.070"/>
   <xacro:property name="wheel_width"  value="0.050"/>
   <xacro:property name="wheel_mass"   value="0.38"/>
-  <xacro:property name="body_mass"    value="8.2"/>
-  <!-- wheel centres in the base frame (axle plane = z 0) -->
-  <xacro:property name="y_corner" value="0.291"/>   <!-- |y| of front/rear wheels -->
-  <xacro:property name="y_mid"    value="0.323"/>   <!-- |y| of middle wheels (wider) -->
-  <xacro:property name="x_front"  value="0.302"/>
-  <xacro:property name="x_mid"    value="0.015"/>
-  <xacro:property name="x_rear"   value="-0.302"/>
+  <xacro:property name="body_mass"    value="6.0"/>
+  <xacro:property name="rocker_mass"  value="0.7"/>
+  <xacro:property name="bogie_mass"   value="0.4"/>
   <material name="body_mat"><color rgba="0.85 0.83 0.78 1.0"/></material>
   <material name="wheel_mat"><color rgba="0.15 0.15 0.17 1.0"/></material>
-  <!-- ===== base / body ===== -->
+  <material name="arm_mat"><color rgba="0.55 0.55 0.58 1.0"/></material>
+  <!-- ===== body ===== -->
   <link name="base_link">
     <visual>
-      <origin xyz="0.05 0 0.251" rpy="0 0 0"/>
+      <origin xyz="0.05 0 0.251"/>
       <geometry><box size="0.555 0.413 0.220"/></geometry>
       <material name="body_mat"/>
     </visual>
     <collision>
-      <origin xyz="0.05 0 0.251" rpy="0 0 0"/>
+      <origin xyz="0.05 0 0.251"/>
       <geometry><box size="0.555 0.413 0.220"/></geometry>
     </collision>
     <inertial>
-      <origin xyz="0.05 0 0.251" rpy="0 0 0"/>
+      <origin xyz="0.05 0 0.251"/>
       <mass value="${body_mass}"/>
-      <inertia ixx="0.150" ixy="0" ixz="0" iyy="0.244" iyz="0" izz="0.327"/>
+      <inertia ixx="0.110" ixy="0" ixz="0" iyy="0.178" iyz="0" izz="0.239"/>
     </inertial>
   </link>
-  <!-- ===== wheel macro (cylinder axis rotated to lie along Y) ===== -->
-  <xacro:macro name="wheel" params="name x y">
+  <!-- ===== a driven wheel (cylinder axis rotated to lie along Y) ===== -->
+  <xacro:macro name="wheel" params="name parent x y z">
     <link name="wheel_${name}">
       <visual>
-        <origin xyz="0 0 0" rpy="1.5708 0 0"/>
+        <origin rpy="1.5708 0 0"/>
         <geometry><cylinder radius="${wheel_radius}" length="${wheel_width}"/></geometry>
         <material name="wheel_mat"/>
       </visual>
       <collision>
-        <origin xyz="0 0 0" rpy="1.5708 0 0"/>
+        <origin rpy="1.5708 0 0"/>
         <geometry><cylinder radius="${wheel_radius}" length="${wheel_width}"/></geometry>
       </collision>
@@ -61,28 +62,56 @@
     </link>
     <joint name="wheel_${name}_joint" type="continuous">
-      <parent link="base_link"/>
+      <parent link="${parent}"/>
       <child link="wheel_${name}"/>
-      <origin xyz="${x} ${y} 0" rpy="0 0 0"/>
+      <origin xyz="${x} ${y} ${z}"/>
       <axis xyz="0 1 0"/>
       <dynamics damping="0.05" friction="0.10"/>
     </joint>
     <gazebo reference="wheel_${name}">
-      <mu1>1.2</mu1>
-      <mu2>1.2</mu2>
-      <kp>1e6</kp>
-      <kd>100.0</kd>
+      <mu1>1.2</mu1><mu2>1.2</mu2><kp>1e6</kp><kd>100.0</kd>
     </gazebo>
   </xacro:macro>
-  <xacro:wheel name="left_front"  x="${x_front}" y="${y_corner}"/>
-  <xacro:wheel name="left_mid"    x="${x_mid}"   y="${y_mid}"/>
-  <xacro:wheel name="left_rear"   x="${x_rear}"  y="${y_corner}"/>
-  <xacro:wheel name="right_front" x="${x_front}" y="${-y_corner}"/>
-  <xacro:wheel name="right_mid"   x="${x_mid}"   y="${-y_mid}"/>
-  <xacro:wheel name="right_rear"  x="${x_rear}"  y="${-y_corner}"/>
-  <!-- ===== ros2_control: a velocity interface on each of the 6 wheels ===== -->
+  <!-- ===== a passive suspension arm (rocker or bogie) ===== -->
+  <xacro:macro name="arm" params="name parent x y z mass len ixx iyy izz">
+    <link name="${name}">
+      <visual>
+        <origin xyz="${len/2 - 0.16} 0 -0.04"/>
+        <geometry><box size="${len} 0.03 0.03"/></geometry>
+        <material name="arm_mat"/>
+      </visual>
+      <inertial>
+        <mass value="${mass}"/>
+        <inertia ixx="${ixx}" ixy="0" ixz="0" iyy="${iyy}" iyz="0" izz="${izz}"/>
+      </inertial>
+    </link>
+    <joint name="${name}_joint" type="revolute">
+      <parent link="${parent}"/>
+      <child link="${name}"/>
+      <origin xyz="${x} ${y} ${z}"/>
+      <axis xyz="0 1 0"/>
+      <limit lower="-0.7" upper="0.7" effort="80" velocity="5"/>
+      <dynamics damping="1.5" friction="0.3"/>
+    </joint>
+  </xacro:macro>
+  <!-- ===== one side: rocker (front wheel) + bogie (mid + rear wheels) ===== -->
+  <xacro:macro name="leg" params="side s">
+    <xacro:arm name="rocker_${side}" parent="base_link"
+               x="0.0" y="${0.27*s}" z="0.12"
+               mass="${rocker_mass}" len="0.45" ixx="0.001" iyy="0.012" izz="0.012"/>
+    <xacro:wheel name="${side}_front" parent="rocker_${side}"
+                 x="0.302" y="${0.021*s}" z="-0.12"/>
+    <xacro:arm name="bogie_${side}" parent="rocker_${side}"
+               x="-0.14" y="${0.03*s}" z="-0.12"
+               mass="${bogie_mass}" len="0.32" ixx="0.0005" iyy="0.0035" izz="0.0035"/>
+    <xacro:wheel name="${side}_mid" parent="bogie_${side}"
+                 x="0.155" y="${0.023*s}" z="0.0"/>
+    <xacro:wheel name="${side}_rear" parent="bogie_${side}"
+                 x="-0.162" y="${-0.009*s}" z="0.0"/>
+  </xacro:macro>
+  <xacro:leg side="left"  s="1"/>
+  <xacro:leg side="right" s="-1"/>
+  <!-- ===== ros2_control: velocity interface on each of the 6 wheels ===== -->
   <ros2_control name="GazeboSimSystem" type="system">
-    <hardware>
-      <plugin>gz_ros2_control/GazeboSimSystem</plugin>
-    </hardware>
+    <hardware><plugin>gz_ros2_control/GazeboSimSystem</plugin></hardware>
     <xacro:macro name="wheel_ctl" params="name">
       <joint name="wheel_${name}_joint">
@@ -99,5 +128,4 @@
     <xacro:wheel_ctl name="right_rear"/>
   </ros2_control>
-  <!-- ===== gz_ros2_control plugin: starts the controller_manager inside Gazebo ===== -->
   <gazebo>
     <plugin filename="gz_ros2_control-system"
@@ -106,9 +134,3 @@
     </plugin>
   </gazebo>
-  <!--
-    TODO (Stage 1 full): replace the rigid wheel mounts with the articulated
-    rocker-bogie — per side: rocker (passive revolute, axis Y) carrying the front
-    wheel + a bogie (passive revolute, axis Y) carrying the mid+rear wheels; add
-    the cross-body differential. Then verify over uneven terrain.
-  -->
 </robot>

Commit message: fix(sim): rename xacro param len->arm_len (builtin clash) + launch on_stderr=ignore
The 'len' macro param shadowed a xacro builtin, emitting a stderr warning that the
launch Command treated as fatal, so the rover never spawned. Rename it and make the
robot_description Command tolerant of benign xacro warnings.

Co-Authored-By: Claude Opus 4.8 <noreply@anthropic.com>

File: src/friday_description/urdf/mark1.urdf.xacro (robot description, xacro)
@@ -73,9 +73,9 @@
   </xacro:macro>
   <!-- ===== a passive suspension arm (rocker or bogie) ===== -->
-  <xacro:macro name="arm" params="name parent x y z mass len ixx iyy izz">
+  <xacro:macro name="arm" params="name parent x y z mass arm_len ixx iyy izz">
     <link name="${name}">
       <visual>
-        <origin xyz="${len/2 - 0.16} 0 -0.04"/>
-        <geometry><box size="${len} 0.03 0.03"/></geometry>
+        <origin xyz="${arm_len/2 - 0.16} 0 -0.04"/>
+        <geometry><box size="${arm_len} 0.03 0.03"/></geometry>
         <material name="arm_mat"/>
       </visual>
@@ -98,10 +98,10 @@
     <xacro:arm name="rocker_${side}" parent="base_link"
                x="0.0" y="${0.27*s}" z="0.12"
-               mass="${rocker_mass}" len="0.45" ixx="0.001" iyy="0.012" izz="0.012"/>
+               mass="${rocker_mass}" arm_len="0.45" ixx="0.001" iyy="0.012" izz="0.012"/>
     <xacro:wheel name="${side}_front" parent="rocker_${side}"
                  x="0.302" y="${0.021*s}" z="-0.12"/>
     <xacro:arm name="bogie_${side}" parent="rocker_${side}"
                x="-0.14" y="${0.03*s}" z="-0.12"
-               mass="${bogie_mass}" len="0.32" ixx="0.0005" iyy="0.0035" izz="0.0035"/>
+               mass="${bogie_mass}" arm_len="0.32" ixx="0.0005" iyy="0.0035" izz="0.0035"/>
     <xacro:wheel name="${side}_mid" parent="bogie_${side}"
                  x="0.155" y="${0.023*s}" z="0.0"/>

Commit message: fix(sim): raise rocker pivot above body CoM so the suspension self-levels
The passive rockers were collapsing to their -0.7 limit (body pitched ~39deg)
because the pivot sat below the body CoM (inverted pendulum). Raise the rocker
pivot to z=0.28 and keep the body CoM low (z=0.18) so the sprung body hangs stably
and self-levels, while the arms still articulate over bumps.

Co-Authored-By: Claude Opus 4.8 <noreply@anthropic.com>

File: src/friday_description/urdf/mark1.urdf.xacro (robot description, xacro)
@@ -39,5 +39,7 @@
     </collision>
     <inertial>
-      <origin xyz="0.05 0 0.251"/>
+      <!-- CoM kept LOW (z=0.18, below the rocker pivots at 0.28) for a stable,
+           self-levelling sprung body — heavy components sit low in the real deck. -->
+      <origin xyz="0.05 0 0.18"/>
       <mass value="${body_mass}"/>
       <inertia ixx="0.110" ixy="0" ixz="0" iyy="0.178" iyz="0" izz="0.239"/>
@@ -96,11 +98,14 @@
   <!-- ===== one side: rocker (front wheel) + bogie (mid + rear wheels) ===== -->
   <xacro:macro name="leg" params="side s">
+    <!-- rocker pivot raised to z=0.28 (ABOVE the body CoM) so the sprung body
+         hangs like a pendulum and self-levels; the arms still articulate over
+         bumps but gravity recenters them. Wheels stay at their measured (x, y). -->
     <xacro:arm name="rocker_${side}" parent="base_link"
-               x="0.0" y="${0.27*s}" z="0.12"
+               x="0.0" y="${0.27*s}" z="0.28"
                mass="${rocker_mass}" arm_len="0.45" ixx="0.001" iyy="0.012" izz="0.012"/>
     <xacro:wheel name="${side}_front" parent="rocker_${side}"
-                 x="0.302" y="${0.021*s}" z="-0.12"/>
+                 x="0.302" y="${0.021*s}" z="-0.28"/>
     <xacro:arm name="bogie_${side}" parent="rocker_${side}"
-               x="-0.14" y="${0.03*s}" z="-0.12"
+               x="-0.14" y="${0.03*s}" z="-0.28"
                mass="${bogie_mass}" arm_len="0.32" ixx="0.0005" iyy="0.0035" izz="0.0035"/>
     <xacro:wheel name="${side}_mid" parent="bogie_${side}"

Commit message: fix(sim): centre body CoM under the rocker pivots (x=0) so it hangs level
Residual ~21deg pitch was the body swinging its forward CoM (x=0.05) under the
pivot line (x=0). Align CoM to x=0 -> hangs level.

Co-Authored-By: Claude Opus 4.8 <noreply@anthropic.com>

File: src/friday_description/urdf/mark1.urdf.xacro (robot description, xacro)
@@ -39,7 +39,8 @@
     </collision>
     <inertial>
-      <!-- CoM kept LOW (z=0.18, below the rocker pivots at 0.28) for a stable,
-           self-levelling sprung body — heavy components sit low in the real deck. -->
-      <origin xyz="0.05 0 0.18"/>
+      <!-- CoM placed UNDER the rocker pivot line (x=0, the pivots' x) and LOW
+           (z=0.18, below the pivots at 0.28) so the sprung body hangs level and
+           self-centres — heavy components sit low and centred in the real deck. -->
+      <origin xyz="0.0 0 0.18"/>
       <mass value="${body_mass}"/>
       <inertia ixx="0.110" ixy="0" ixz="0" iyy="0.178" iyz="0" izz="0.239"/>
