Commit message: fix(description): lidar rides the mast head; arena furniture raised to match
With the real chassis mesh the old lidar mount (0.05,0,0.25) sat INSIDE
the body: 2720 self-return triangles boxed the costmap in and Nav2
could not plan at all (found by the isolated phase-3 gate — planner
'Failed to create plan', behaviors 'Collision Ahead'). The lidar now
mounts on the camera-mast head (0.193,-0.101,0.57), above every body
part (mesh top 0.544, antenna 0.414) — which is the actual Mark 1 plan
for the mast. Scan plane is now 0.64 m above ground, so arena walls go
0.6->1.2 m, pillars 0.5->0.9 m, crate 0.4->0.8 m. maps/arena is stale
(recorded from the old scan height); demos run live SLAM, regenerate
when needed.

Co-Authored-By: Claude Opus 4.8 <noreply@anthropic.com>

File: src/friday_description/urdf/mark1.urdf.xacro (robot description, xacro)
@@ -140,5 +140,9 @@
   <joint name="lidar_joint" type="fixed">
     <parent link="base_link"/><child link="lidar_link"/>
-    <origin xyz="0.05 0 0.25" rpy="0 0 0"/>
+    <!-- mast-head mount (the replica's camera mast carries Mark 1's sensors):
+         above the whole body mesh, so the lidar never sees its own chassis.
+         At the old 0.25 height the real body boxed the scan in — 2720
+         self-return triangles -> costmap lethal ring -> Nav2 could not plan. -->
+    <origin xyz="0.193 -0.101 0.57" rpy="0 0 0"/>
   </joint>
   <link name="imu_link">

Commit message: feat(sim): 3D perception -> fused voxel world for the Command Center
The 2D /scan can't see height, so the deck could only draw a floor-plan.
This gives the sim real 3D eyes and streams the reconstruction:

- URDF: a 16-ring 3D lidar (360deg, +/-15deg) + a forward depth camera
  on the mast. Verified: 2880 + 19200 points/frame.
- telemetry agent fuses both clouds into an accumulating MAP-FRAME voxel
  world (10 cm cubes), floor/ceiling clipped, capped at 24k voxels
  (LRU-evicted), and streams it as signed tlm/voxel: int16 triplets,
  zlib+b64, digest-gated on growth, 256 KB refuse-ceiling. Whole 8x8
  arena world = ~7.4k voxels in a 22 KB signed envelope.

Two bugs fixed on the way, both found live:
- CLOCK DOMAIN: the agent keeps WALL clock (envelope expiry) but sim TF
  is stamped in SIM time -> a wall-clock buffer evicted every transform
  as ancient, so map->base_link and map->sensor lookups silently failed.
  THIS is why the rover rendered outside its own walls (pose fell back
  to dead-reckon). Fix: a dedicated TF sub-node on its own clock
  (tf_use_sim_time:=true in sim), leaving the authority logic on wall
  time. Odom now radios the true map-frame pose.
- depth sensors emit NaN/inf for invalid returns; int(NaN) crashed the
  voxelizer (killed the agent). Finite-guard in the pure add_points.

144 tests green.

Co-Authored-By: Claude Opus 4.8 <noreply@anthropic.com>

File: src/friday_description/urdf/mark1.urdf.xacro (robot description, xacro)
@@ -178,3 +178,56 @@
     </sensor>
   </gazebo>
+  <!-- ===== 3D perception (sim stand-ins for the Research Deck) =====
+       A 16-ring 3D lidar (360deg, +/-15deg) + a forward depth camera, both on
+       the mast. They see HEIGHT, which the 2D /scan cannot — the raw material
+       for the Command Center's true-3D environment reconstruction. Clouds are
+       fused + voxelized + streamed by the telemetry agent, never raw to the CC
+       (data-gate rule). -->
+  <link name="lidar3d_link">
+    <inertial><mass value="0.1"/>
+      <inertia ixx="1e-4" iyy="1e-4" izz="1e-4" ixy="0" ixz="0" iyz="0"/></inertial>
+  </link>
+  <joint name="lidar3d_joint" type="fixed">
+    <parent link="base_link"/><child link="lidar3d_link"/>
+    <origin xyz="0.193 -0.101 0.60" rpy="0 0 0"/>
+  </joint>
+  <gazebo reference="lidar3d_link">
+    <sensor name="lidar3d" type="gpu_lidar">
+      <topic>lidar3d</topic>
+      <gz_frame_id>lidar3d_link</gz_frame_id>
+      <update_rate>8</update_rate>
+      <lidar>
+        <scan>
+          <horizontal><samples>180</samples><resolution>1</resolution>
+            <min_angle>-3.14159</min_angle><max_angle>3.14159</max_angle></horizontal>
+          <vertical><samples>16</samples><resolution>1</resolution>
+            <min_angle>-0.262</min_angle><max_angle>0.262</max_angle></vertical>
+        </scan>
+        <range><min>0.2</min><max>12.0</max><resolution>0.01</resolution></range>
+      </lidar>
+      <always_on>true</always_on><visualize>false</visualize>
+    </sensor>
+  </gazebo>
+  <link name="depthcam_link">
+    <inertial><mass value="0.05"/>
+      <inertia ixx="1e-5" iyy="1e-5" izz="1e-5" ixy="0" ixz="0" iyz="0"/></inertial>
+  </link>
+  <joint name="depthcam_joint" type="fixed">
+    <!-- forward-looking on the mast; optical frame handled via TF downstream -->
+    <parent link="base_link"/><child link="depthcam_link"/>
+    <origin xyz="0.28 -0.101 0.52" rpy="0 0 0"/>
+  </joint>
+  <gazebo reference="depthcam_link">
+    <sensor name="depthcam" type="depth_camera">
+      <topic>depthcam</topic>
+      <gz_frame_id>depthcam_link</gz_frame_id>
+      <update_rate>8</update_rate>
+      <camera>
+        <horizontal_fov>1.3</horizontal_fov>
+        <image><width>160</width><height>120</height></image>
+        <clip><near>0.1</near><far>10.0</far></clip>
+      </camera>
+      <always_on>true</always_on><visualize>false</visualize>
+    </sensor>
+  </gazebo>
 </robot>

Commit message: wip(rover): mission executor + GPS + navsat + mission planner (unfinished)
Preserving in-progress work from the rover-mission-executor agent (hit
session limit mid-retry-logic). Rover-side additions:

  * friday_telemetry/geo.py — WGS84 <-> map-frame helpers
  * friday_telemetry/mission_planner.py — lawnmower survey plan_survey()
  * telemetry_agent_node.py — mission executor state machine (dedicated
    callback group, MECE with vitals; enqueue-and-drain pattern);
    tlm/mission progress publisher
  * sim_os.launch.py + urdf + navsat_transform.yaml — GPS sensor + the
    utm->map anchor
  * nav2.yaml — tuning for outdoor SLAM
  * baylands.sdf — nav markers

Known gap: waypoint failed 30 retries when the survey zone corner falls
outside the current SLAM map (planner rejects OOB coords). Retry logic
still being iterated. Currently running in memory in the live demo
container.

Co-Authored-By: Claude Fable 5 <noreply@anthropic.com>

File: src/friday_description/urdf/mark1.urdf.xacro (robot description, xacro)
@@ -231,3 +231,30 @@
     </sensor>
   </gazebo>
+  <!-- ===== GPS / NavSat (sim stand-in for the rover's GPS module) =====
+       Baylands world carries real WGS84 spherical coordinates (lat 37.41 N,
+       lon -121.99 W) so the NavSat sensor reports genuine lat/lon for this
+       location. The bridge maps gz topic /gps/fix -> ROS /gps/fix (NavSatFix)
+       so the telemetry agent can forward it to the FCC and navsat_transform
+       can anchor the map frame to the real-world position. -->
+  <link name="gps_link">
+    <inertial><mass value="0.02"/>
+      <inertia ixx="1e-5" iyy="1e-5" izz="1e-5" ixy="0" ixz="0" iyz="0"/></inertial>
+  </link>
+  <joint name="gps_joint" type="fixed">
+    <parent link="base_link"/><child link="gps_link"/>
+    <origin xyz="0 0 0.40" rpy="0 0 0"/>
+  </joint>
+  <gazebo reference="gps_link">
+    <sensor name="gps" type="navsat">
+      <topic>gps/fix</topic>
+      <update_rate>1</update_rate>
+      <always_on>true</always_on>
+      <navsat>
+        <position_sensing>
+          <horizontal><noise type="gaussian"><mean>0</mean><stddev>0.0001</stddev></noise></horizontal>
+          <vertical><noise type="gaussian"><mean>0</mean><stddev>0.0002</stddev></noise></vertical>
+        </position_sensing>
+      </navsat>
+    </sensor>
+  </gazebo>
 </robot>

Commit message: feat(sim): bumper-height ground-scan RGB-D sensor for terrain intelligence
Adds a 128×96 downward-tilted (30°) RGB-D depth camera at the front
bumper (x=0.32, z=0.14, front of the front axle). Where the mast lidar
sees the TOP of a slope (registers as wall in Nav2's flat costmap), this
sensor sees the SURFACE ahead of the wheels. Downstream terrain
classifier will use it to distinguish 'climbable slope' from 'vertical
wall'.

Sensor: gpu rgbd_camera, 10 Hz target, FOV 60°, near 5 cm, far 3 m.
Fixed joint to base_link (no articulation). Bridged as
/ground_scan/points (PointCloud2, gz.msgs.PointCloudPacked).

Verified live: /ground_scan/points publishing at 4.7 Hz, 12288 dense
points per frame, XYZRGB packed. Sim spawns clean, no controller or
Gazebo errors.

First of four commits building terrain-intelligence: sensor, classifier,
Nav2 layer, deck overlay.

Co-Authored-By: Claude Fable 5 <noreply@anthropic.com>

File: src/friday_description/urdf/mark1.urdf.xacro (robot description, xacro)
@@ -231,4 +231,34 @@
     </sensor>
   </gazebo>
+  <!-- ===== bumper-height ground-scan RGB-D (terrain intelligence) =====
+       Downward-tilted depth camera at the front bumper. Where the mast lidar
+       sees the TOP of a slope (registers as wall in the flat costmap), this
+       sensor sees the SURFACE ahead of the wheels — so the terrain classifier
+       can tell "climbable slope" from "vertical wall". Short range (max 3 m),
+       narrow-mounted (128×96) so the classifier stays cheap. -->
+  <link name="ground_scan_link">
+    <inertial><mass value="0.05"/>
+      <inertia ixx="1e-5" iyy="1e-5" izz="1e-5" ixy="0" ixz="0" iyz="0"/></inertial>
+  </link>
+  <joint name="ground_scan_joint" type="fixed">
+    <parent link="base_link"/><child link="ground_scan_link"/>
+    <!-- x=0.32: forward of front axle so wheels don't occlude the scan.
+         z=0.14: just above the wheels (wheel top ~0.134 m).
+         pitch=0.524 rad (30°): nose down for a ~0.4-1.5 m ground swath. -->
+    <origin xyz="0.32 0 0.14" rpy="0 0.524 0"/>
+  </joint>
+  <gazebo reference="ground_scan_link">
+    <sensor name="ground_scan" type="rgbd_camera">
+      <topic>ground_scan</topic>
+      <gz_frame_id>ground_scan_link</gz_frame_id>
+      <update_rate>10</update_rate>
+      <camera>
+        <horizontal_fov>1.05</horizontal_fov>
+        <image><width>128</width><height>96</height></image>
+        <clip><near>0.05</near><far>3.0</far></clip>
+      </camera>
+      <always_on>true</always_on><visualize>false</visualize>
+    </sensor>
+  </gazebo>
   <!-- ===== GPS / NavSat (sim stand-in for the rover's GPS module) =====
        Baylands world carries real WGS84 spherical coordinates (lat 37.41 N,
